Commit message: EUH-1 v1: ankle-roll reclassed C->B per R1 verdict (+1.3 kg, 31.88 kg total)
Class counts now derived from joint defs (6A/9B/8C). Stand+pushes revalidated.

Co-Authored-By: Claude Fable 5 <noreply@anthropic.com>

File: sim/model/euh1.urdf (robot description, URDF)
Before this commit: robot euh1, 24 links, 23 joints
Links:
- link left_foot: mass 0.71 -> 1.36
- link right_foot: mass 0.71 -> 1.36
Joints:
- joint left_ankle_roll: limit lower=-0.523599 upper=0.523599 effort=20 velocity=26 -> lower=-0.523599 upper=0.523599 effort=48 velocity=20.4
- joint right_ankle_roll: limit lower=-0.523599 upper=0.523599 effort=20 velocity=26 -> lower=-0.523599 upper=0.523599 effort=48 velocity=20.4
